File: schem/kozo.sch (KiCad schematic (older format))
At the start: 16 parts

Commit message: basic layout
Parts:
- added C3: 1u0/35V, Capacitors_SMD:C_1206, symbol Device:C_Small
- added C4, C5: 100n, Capacitors_SMD:C_0603, symbol Device:C_Small
- added D1: UniTSV, Diodes_SMD:D_SMA, symbol my_device:UniTSV
- J1: renamed from J?; footprint (none) -> PA257-508:PA257_508_02
- J2, J4: renamed from J?; footprint (none) -> Pin_Headers:Pin_Header_Straight_1x03_Pitch2.54mm
- J3: renamed from J?; footprint (none) -> PA257-508:PA257_508_06
- J5: renamed from J?; footprint (none) -> PA357-381:PA357_381_04
- RV1: renamed from RV?; footprint (none) -> Potentiometers:Potentiometer_Trimmer-EVM3E
- U1: renamed from U?; footprint Package_TO_SOT_SMD:SOT-89-3 -> TO_SOT_Packages_SMD:SOT-89-3
- U2: renamed from U?; footprint Package_SO:TSSOP-14_4.4x5mm_P0.65mm -> Housings_SSOP:TSSOP-14_4.4x5mm_Pitch0.65mm
- gave numbers to parts that had none: 8
Connections:
- net +3V3: now also C4.1, C5.1
- net GND: now also C3.2, C4.2, C5.2, D1.2 (A)
- net at J1.2 (Pin_2), U1.3 (IN): now also C3.1, D1.1 (K)
Other:
- moved on the sheet: C1, J1, U1

Commit message: silkscreen
Parts:
- renumbered U2 to IC1, U1 to IC2, J5 to J2, J4 to J3, J3 to J4, J2 to X1
Changed lines of the file:
@@
 $EndDescr
 $Comp
-L MCU_Texas_MSP430:MSP430G2231IPW14 U2
+L MCU_Texas_MSP430:MSP430G2231IPW14 IC1
 U 1 1 5EFEB83B
 P 5000 4650
-F 0 "U2" H 5000 5631 50  0000 C CNN
+F 0 "IC1" H 5000 5631 50  0000 C CNN
 F 1 "MSP430G2231IPW14" H 5450 5400 50  0000 C CNN
 F 2 "Housings_SSOP:TSSOP-14_4.4x5mm_Pitch0.65mm" H 4300 4000 50  0001 C CIN
@@
 $EndComp
 $Comp
-L Regulator_Linear:L78L33_SOT89 U1
+L Regulator_Linear:L78L33_SOT89 IC2
 U 1 1 5EFF363F
 P 3100 2100
-F 0 "U1" H 3100 2342 50  0000 C CNN
+F 0 "IC2" H 3100 2342 50  0000 C CNN
 F 1 "L78L33_SOT89" H 3100 2251 50  0000 C CNN
 F 2 "TO_SOT_Packages_SMD:SOT-89-3" H 3100 2300 50  0001 C CIN
@@
 BACKWARD\nFORWARD\nRELEASE\nGND
 $Comp
-L Connector_Generic:Conn_01x04 J5
+L Connector_Generic:Conn_01x04 J2
 U 1 1 5F03D693
 P 8800 4650
-F 0 "J5" H 8718 4225 50  0000 C CNN
+F 0 "J2" H 8718 4225 50  0000 C CNN
 F 1 "Conn_01x04" H 8718 4316 50  0000 C CNN
 F 2 "PA357-381:PA357_381_04" H 8800 4650 50  0001 C CNN
@@
 $EndComp
 $Comp
-L Connector_Generic:Conn_01x03 J4
+L Connector_Generic:Conn_01x03 J3
 U 1 1 5F03DE39
 P 8800 4050
-F 0 "J4" H 8880 4092 50  0000 L CNN
+F 0 "J3" H 8880 4092 50  0000 L CNN
 F 1 "Conn_01x03" H 8880 4001 50  0000 L CNN
 F 2 "Pin_Headers:Pin_Header_Straight_1x03_Pitch2.54mm" H 8800 4050 50  0001 C CNN
@@
 	6550 3750 6550 3850
 $Comp
-L Connector_Generic:Conn_01x06 J3
+L Connector_Generic:Conn_01x06 J4
 U 1 1 5F057126
 P 8800 3450
-F 0 "J3" H 8718 2925 50  0000 C CNN
+F 0 "J4" H 8718 2925 50  0000 C CNN
 F 1 "Conn_01x06" H 8718 3016 50  0000 C CNN
 F 2 "PA257-508:PA257_508_06" H 8800 3450 50  0001 C CNN
@@
 	8500 3550 8500 3950
 $Comp
-L Connector_Generic:Conn_01x03 J2
+L Connector_Generic:Conn_01x03 X1
 U 1 1 5F060DB8
 P 6050 3450
-F 0 "J2" V 6014 3262 50  0000 R CNN
+F 0 "X1" V 6014 3262 50  0000 R CNN
 F 1 "Conn_01x03" V 5923 3262 50  0000 R CNN
 F 2 "Pin_Headers:Pin_Header_Straight_1x03_Pitch2.54mm" H 6050 3450 50  0001 C CNN

Commit message: nice schmatic
Parts:
- D1: value UniTSV -> SMAJ33A
Other:
- note added: "+24V\nGND"
Changed lines of the file:
@@
 U 1 1 5EFEB83B
 P 5000 4650
-F 0 "IC1" H 5000 5631 50  0000 C CNN
+F 0 "IC1" H 4300 5400 50  0000 C CNN
 F 1 "MSP430G2231IPW14" H 5450 5400 50  0000 C CNN
 F 2 "Housings_SSOP:TSSOP-14_4.4x5mm_Pitch0.65mm" H 4300 4000 50  0001 C CIN
@@
 U 1 1 5EFEC8F1
 P 3950 4000
-F 0 "R1" H 4009 4046 50  0000 L CNN
-F 1 "10k" H 4009 3955 50  0000 L CNN
+F 0 "R1" H 3750 4100 50  0000 L CNN
+F 1 "10k" H 3750 3950 50  0000 L CNN
 F 2 "Resistors_SMD:R_0603" H 3950 4000 50  0001 C CNN
 F 3 "~" H 3950 4000 50  0001 C CNN
@@
 U 1 1 5EFF0E73
 P 7350 5300
-F 0 "C2" H 7442 5346 50  0000 L CNN
-F 1 "100n" H 7442 5255 50  0000 L CNN
+F 0 "C2" H 7100 5350 50  0000 L CNN
+F 1 "100n" H 7050 5250 50  0000 L CNN
 F 2 "Capacitors_SMD:C_0603" H 7350 5300 50  0001 C CNN
 F 3 "~" H 7350 5300 50  0001 C CNN
@@
 U 1 1 5EFF8ABB
 P 1400 2200
-F 0 "J1" H 1318 1875 50  0000 C CNN
-F 1 "Conn_01x02" H 1318 1966 50  0000 C CNN
+F 0 "J1" H 1400 2000 50  0000 C CNN
+F 1 "Conn_01x02" H 1318 1966 50  0001 C CNN
 F 2 "PA257-508:PA257_508_02" H 1400 2200 50  0001 C CNN
 F 3 "~" H 1400 2200 50  0001 C CNN
@@
 U 1 1 5F000254
 P 6350 3950
-F 0 "R2" H 6409 3996 50  0000 L CNN
-F 1 "10k" H 6409 3905 50  0000 L CNN
+F 0 "R2" H 6200 4100 50  0000 L CNN
+F 1 "10k" H 6350 3800 50  0000 L CNN
 F 2 "Resistors_SMD:R_0603" H 6350 3950 50  0001 C CNN
 F 3 "~" H 6350 3950 50  0001 C CNN
@@
 U 1 1 5F000AE7
 P 6550 3950
-F 0 "R3" H 6609 3996 50  0000 L CNN
-F 1 "10k" H 6609 3905 50  0000 L CNN
+F 0 "R3" H 6400 4100 50  0000 L CNN
+F 1 "10k" H 6600 3800 50  0000 L CNN
 F 2 "Resistors_SMD:R_0603" H 6550 3950 50  0001 C CNN
 F 3 "~" H 6550 3950 50  0001 C CNN
@@
 U 1 1 5F000D13
 P 6750 3950
-F 0 "R4" H 6809 3996 50  0000 L CNN
-F 1 "10k" H 6809 3905 50  0000 L CNN
+F 0 "R4" H 6600 4100 50  0000 L CNN
+F 1 "10k" H 6800 3800 50  0000 L CNN
 F 2 "Resistors_SMD:R_0603" H 6750 3950 50  0001 C CNN
 F 3 "~" H 6750 3950 50  0001 C CNN
@@
 U 1 1 5F03D693
 P 8800 4650
-F 0 "J2" H 8718 4225 50  0000 C CNN
-F 1 "Conn_01x04" H 8718 4316 50  0000 C CNN
+F 0 "J2" H 8800 4350 50  0000 C CNN
+F 1 "Conn_01x04" H 8718 4316 50  0001 C CNN
 F 2 "PA357-381:PA357_381_04" H 8800 4650 50  0001 C CNN
 F 3 "~" H 8800 4650 50  0001 C CNN
@@
 U 1 1 5F03DE39
 P 8800 4050
-F 0 "J3" H 8880 4092 50  0000 L CNN
-F 1 "Conn_01x03" H 8880 4001 50  0000 L CNN
+F 0 "J3" H 8750 4250 50  0000 L CNN
+F 1 "Conn_01x03" H 8880 4001 50  0001 L CNN
 F 2 "Pin_Headers:Pin_Header_Straight_1x03_Pitch2.54mm" H 8800 4050 50  0001 C CNN
 F 3 "~" H 8800 4050 50  0001 C CNN
@@
 P 6750 3750
 F 0 "#PWR0112" H 6750 3600 50  0001 C CNN
-F 1 "+3V3" H 6765 3923 50  0000 C CNN
+F 1 "+3V3" H 6550 3950 50  0000 C CNN
 F 2 "" H 6750 3750 50  0001 C CNN
 F 3 "" H 6750 3750 50  0001 C CNN
@@
 P 6550 3750
 F 0 "#PWR0113" H 6550 3600 50  0001 C CNN
-F 1 "+3V3" H 6565 3923 50  0000 C CNN
+F 1 "+3V3" H 6550 3950 50  0000 C CNN
 F 2 "" H 6550 3750 50  0001 C CNN
 F 3 "" H 6550 3750 50  0001 C CNN
@@
 P 6350 3750
 F 0 "#PWR0114" H 6350 3600 50  0001 C CNN
-F 1 "+3V3" H 6365 3923 50  0000 C CNN
+F 1 "+3V3" H 6550 3950 50  0000 C CNN
 F 2 "" H 6350 3750 50  0001 C CNN
 F 3 "" H 6350 3750 50  0001 C CNN
@@
 U 1 1 5F057126
 P 8800 3450
-F 0 "J4" H 8718 2925 50  0000 C CNN
-F 1 "Conn_01x06" H 8718 3016 50  0000 C CNN
+F 0 "J4" H 8800 3050 50  0000 C CNN
+F 1 "Conn_01x06" H 8718 3016 50  0001 C CNN
 F 2 "PA257-508:PA257_508_06" H 8800 3450 50  0001 C CNN
 F 3 "~" H 8800 3450 50  0001 C CNN
@@
 U 1 1 5F060DB8
 P 6050 3450
-F 0 "X1" V 6014 3262 50  0000 R CNN
-F 1 "Conn_01x03" V 5923 3262 50  0000 R CNN
+F 0 "X1" V 6150 3700 50  0000 R CNN
+F 1 "Conn_01x03" V 6150 3650 50  0001 R CNN
 F 2 "Pin_Headers:Pin_Header_Straight_1x03_Pitch2.54mm" H 6050 3450 50  0001 C CNN
 F 3 "~" H 6050 3450 50  0001 C CNN
@@
 P 1900 2300
 F 0 "D1" H 1968 2330 40  0000 L CNN
-F 1 "UniTSV" H 1968 2262 30  0000 L CNN
+F 1 "SMAJ33A" H 1968 2262 30  0000 L CNN
 F 2 "Diodes_SMD:D_SMA" H 1968 2232 60  0001 L CNN
 F 3 "" V 1800 2310 60  0000 C CNN
@@
 Wire Wire Line
 	1900 2400 1900 2500
+Text Notes 1300 2250 2    63   ~ 0
++24V\nGND
 $EndSCHEMATC
