File: schem/kozo.kicad_pcb (KiCad board)
At the start: 2 copper layers, 38.7 x 20.3 mm, 20 parts, among them J1 Conn_01x02, J2 Conn_01x03, J3 Conn_01x06, J4 Conn_01x03, J5 Conn_01x04, U1 L78L33_SOT89, U2 MSP430G2231IPW14

Commit message: layout
Parts:
- moved C1 0.64 mm to (154.9, 102.2)
- moved C2 0.64 mm to (177.8, 101.6)
- moved C3 0.64 mm to (154.9, 112.4)
- moved C4 0.64 mm to (168.3, 107.3)
- moved C5 0.64 mm to (177.8, 113.0)
- moved D1 0.64 mm to (150.5, 107.3)
- moved J1 0.64 mm to (146.1, 107.3)
- moved J3 0.64 mm to (162.6, 98.4)
- moved J5 0.64 mm to (167.0, 112.4)
- moved R2 0.64 mm to (171.4, 109.2)
- moved R3 0.64 mm to (168.3, 109.2)
- moved R4 0.64 mm to (165.1, 109.2)
- moved R5 0.64 mm to (175.3, 109.2)
- moved R6 0.64 mm to (174.6, 101.6)
- moved RV1 0.64 mm to (175.3, 105.4)
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Routing:
- net GND: track 0.00 -> 86.4 mm, vias 0 -> 23
- net +3V3: track 21.2 -> 77.0 mm, vias 0 -> 3
- net Net-(J3-Pad1): track 0.00 -> 27.9 mm, vias 0 -> 1
- net Net-(C2-Pad1): track 17.7 -> 16.5 mm, vias 1 -> 0
- net Net-(J5-Pad4): track 15.3 -> 15.9 mm
- net Net-(J5-Pad3): track 15.7 -> 16.3 mm
- added copper zone on B.Cu, net GND
- added copper zone on F.Cu, net GND
Other:
- board size 38.7 x 20.3 mm -> 40.6 x 22.9 mm
- net class D04 added: clearance 0.2, trace_width 0.4, via_dia 0.8, via_drill 0.4
- board text added: "+"
- board text added: "-"
- board text added: "202007 OH"
- board text added: "24V"
- board text added: "BCK"
- board text added: "DIR"
- board text added: "ENA"
- board text added: "FWD"
- board text added: "GND"
- board text added: "PUL"
- board text added: "REL"
- board text added: "SPD"
- board text added: "https://github.com/ondrejh/kozopec"

Commit message: silkscreen
Parts:
- renumbered U2 to IC1, U1 to IC2, J5 to J2, J4 to J3, J3 to J4, J2 to X1

Commit message: silk goat
Parts:
- added LOGO: , schem:koza, F.Cu at (177.8, 95.9)
- added LOGO: , schem:koza_inv, F.Cu at (143.5, 95.9)
- D1: value UniTSV -> SMAJ33A
Other:
- board text added: "2020.07 OH"
- board text added: "https://github.com/ ondrejh/kozopec"
- board text removed: "202007 OH"

Commit message: mask debug
Routing:
- net +3V3: track 77.0 -> 78.3 mm
